Commit message: Add stl file of set, but glasses are not included

File: room/set.urdf (robot description, URDF)
Before this commit: robot set, 1 links, 0 joints
Links:
- added link obstacle_base_bis; collision mesh filename=package://iai_maps/meshes/set_wine.stl; visual mesh filename=package://iai_maps/meshes/set_wine.dae
Joints:
- added joint j_obstacle_base_bis: type fixed, parent obstacle_base, child obstacle_base_bis, origin xyz=0 0 0 rpy=0 0 0
