Commit message: change room floor stuff

File: room/floor.urdf (robot description, URDF)
Before this commit: robot floor, 3 links, 2 joints
Links:
- link l_floor: geometry collision box size=10 10 0.005; visual box size=10 10 0.005
- link l_wall: geometry collision box size=10 0.005 2; visual box size=10 0.005 2
- link obstacle_base: geometry visual box size=0.001 0.001 0.001
