Commit message: Location changes in kitchen with flowers and chair

File: room/chair.urdf (robot description, URDF)
Before this commit: robot chair, 1 links, 0 joints
Links:
- link obstacle_base: geometry collision mesh filename=package://iai_maps/meshes/high_chair_placed.stl; visual mesh filename=package://iai_maps/meshes/high_chair_placed.stl

File: room/floor.urdf (robot description, URDF)
Before this commit: robot floor, 3 links, 2 joints
Links:
- link l_floor: geometry collision box size=10 10 0.005; visual box size=10 14 0.005

File: room/flower-vase.urdf (robot description, URDF)
Before this commit: robot flowers, 1 links, 0 joints
Links:
- link obstacle_base: geometry collision box size=0.4 0.4 0.4; visual mesh filename=package://iai_maps/meshes/flower-vase.dae

File: room/set.urdf (robot description, URDF)
Before this commit: robot set, 2 links, 1 joints
Links:
- removed link obstacle_base_bis
- link obstacle_base: geometry collision mesh filename=package://iai_maps/meshes/set_wine.stl; visual mesh filename=package://iai_maps/meshes/set_wine.stl
Joints:
- removed joint j_obstacle_base_bis
